File: Rocket_v1.kicad_pcb (KiCad board)
At the start: 2 copper layers, 3 parts

Commit message: Add files via upload
Parts:
- added Mosfet1: ~, AAABryces_lib:Mosfet, F.Cu at (68.5, 49.1)
- added Screw1: ~, AAABryces_lib:2 pin Screw term, F.Cu at (76.6, 29.0)
Connections:
- ESP1 pad 6: unconnected-(ESP1-26-Pad6) -> Net-(ESP1-26)
Routing:
- net Net-(ESP1-26): track 0.00 -> 35.5 mm
- net Net-(Mosfet1-Drain): track 0.00 -> 9.25 mm
- net Net-(Mosfet1-Source): track 0.00 -> 8.46 mm
- net Net-(HX1-GND): track 31.8 -> 29.6 mm
- net Net-(ESP1-VIN): track 32.2 -> 31.2 mm
