File: Rocket_v1.kicad_sch (KiCad schematic)
At the start: 5 parts

Commit message: Add files via upload
Changed lines of the file:
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@@
     )
   )
-  (symbol (lib_name "HX711_Bryce_1") (lib_id "AAABryces_symbols:HX711_Bryce") (at 207.01 80.01 180) (unit 1)
+  (symbol (lib_id "AAABryces_symbols:HX711_Bryce") (at 207.01 80.01 180) (unit 1)
     (in_bom yes) (on_board yes) (dnp no) (fields_autoplaced)
     (property "Reference" "HX1" (at 200.66 64.77 0)
@@
       (effects (font (size 1.27 1.27)) hide)
     )
-    (pin "3")
     (pin "5")
     (pin "8")
     (pin "7")
-    (pin "4")
-    (pin "2")
     (pin "6")
-    (pin "1")
     (instances
       (project "Rocket_v1"
